Commit message: added jodell RG52-050 gripper support

File: fairino5_v6_moveit2_config/config/fairino5_v6_robot.ros2_control.xacro (robot description, xacro)
@@ -2,5 +2,5 @@
 <robot xmlns:xacro="http://www.ros.org/wiki/xacro">
     <xacro:macro name="fairino5_v6_robot_ros2_control" params="name initial_positions_file">
-        <xacro:property name="initial_positions" value="${load_yaml(initial_positions_file)['initial_positions']}"/>
+        <xacro:property name="initial_positions" value="${xacro.load_yaml(initial_positions_file)['initial_positions']}"/>
         <ros2_control name="${name}" type="system">
             <hardware>
@@ -8,4 +8,14 @@
                 <!--<plugin>mock_components/GenericSystem</plugin>-->
                 <plugin>fairino_hardware/FairinoHardwareInterface</plugin>
+                <!-- Gripper configuration parameters -->
+                <param name="gripper_company">6</param>
+                <param name="gripper_device">0</param>
+                <param name="gripper_softversion">0</param>
+                <param name="gripper_bus">1</param>
+                <param name="gripper_index">1</param>
+                <param name="gripper_max_time">5000</param>
+                <param name="gripper_position_tolerance">0.001</param>
+                <param name="gripper_max_velocity">50.0</param>
+                <param name="gripper_max_effort">50.0</param>
             </hardware>
             <joint name="j1">
@@ -45,4 +55,21 @@
                 </state_interface>
             </joint>
+            <!-- Gripper joints -->
+            <joint name="left_finger_joint">
+                <command_interface name="position"/>
+                <state_interface name="position">
+                  <param name="initial_value">0.0</param>
+                </state_interface>
+                <state_interface name="velocity"/>
+                <state_interface name="effort"/>
+            </joint>
+            <!-- Right finger joint is a mimic joint - only add state interfaces for simulation/visualization -->
+            <joint name="right_finger_joint">
+                <state_interface name="position">
+                  <param name="initial_value">0.0</param>
+                </state_interface>
+                <state_interface name="velocity"/>
+                <state_interface name="effort"/>
+            </joint>
         </ros2_control>
     </xacro:macro>

File: fairino_description/urdf/fairino5_v6.urdf (robot description, URDF)
Before this commit: robot fairino5_v6_robot, 7 links, 6 joints
Links:
- added link gripper_base_link, mass 1.0; collision mesh filename=package://fairino_description/meshes/fairino5_v6/gripper_ba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; visual mesh filename=package://fairino_description/meshes/fairino5_v6/gripper_ba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
- added link left_finger, mass 0.1; collision mesh filename=package://fairino_description/meshes/fairino5_v6/left_grip.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 scale=0.001 0.001 0.001; visual mesh filename=package://fairino_description/meshes/fairino5_v6/left_grip.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 scale=0.001 0.001 0.001
- added link right_finger, mass 0.1; collision mesh filename=package://fairino_description/meshes/fairino5_v6/right_grip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 scale=0.001 0.001 0.001; visual mesh filename=package://fairino_description/meshes/fairino5_v6/right_grip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 scale=0.001 0.001 0.001
Joints:
- added joint gripper_joint: type fixed, parent wrist3_link, child gripper_base_link, origin xyz=0 0 0.08 rpy=0 0 0
- added joint left_finger_joint: type prismatic, parent gripper_base_link, child left_finger, origin xyz=-0.016 0.009 0.10225 rpy=0 0 0, axis 1 0 0, limit lower=0.0 upper=0.01825 effort=50 velocity=1.0
- added joint right_finger_joint: type prismatic, parent gripper_base_link, child right_finger, origin xyz=0.016 -0.009 0.10225 rpy=0 0 0, axis -1 0 0, limit lower=0.0 upper=0.01825 effort=50 velocity=1.0, mimic joint=left_finger_joint
